File: hardware/KiCad - node V2/RP2350.kicad_pcb (KiCad board)
At the start: 4 copper layers, 145.6 x 52 mm, 86 parts, among them J3 USB_C_Receptacle_USB2.0_14P, SW1 BOOTSEL, U1 RP2350A, U2 THVD1450D, U3 ADXL355BEZ, U4 TPS2121RUXR, U5 USBLC6-2SC6, U6 TLV75733PDBV, U7 W25Q128JVS, U8 TPS7A20xxxDBV

Commit message: hardware: new layout
Parts:
- removed R11: 0 DNP, Resistor_SMD:R_0805_2012Metric
- removed R25, R26, R28, R29: 33ohm, Resistor_SMD:R_0603_1608Metric
- added REF**: MountingHole_2.5mm, MountingHole:MountingHole_2.5mm, F.Cu at (156.9, 35.8)
- added REF**: MountingHole_2.5mm, MountingHole:MountingHole_2.5mm, F.Cu at (176.9, 35.8)
- C30, C34, C35, C37: footprint Capacitor_SMD:C_0603_1608Metric -> Capacitor_SMD:C_0402_1005Metric
- C36: footprint Capacitor_SMD:C_0805_2012Metric -> Capacitor_SMD:C_0603_1608Metric
- R23, R24, R27: footprint Resistor_SMD:R_0603_1608Metric -> Resistor_SMD:R_0402_1005Metric
- moved C24 91.0 mm to (152.8, 32.3), turned to 90 degrees
- moved R20 71.4 mm to (149.4, 22.9), turned to 90 degrees
- moved D3 71.3 mm to (151.1, 22.9), turned to -90 degrees
- moved C15 61.0 mm to (146.3, 22.6)
- moved C16 61.0 mm to (143.2, 26.5)
- moved C17 61.0 mm to (143.4, 28.6)
- moved C18 61.0 mm to (143.2, 30.8)
- moved U6 61.0 mm to (143.2, 23.0)
- moved C14 52.2 mm to (172.0, 21.7), turned to 90 degrees
- moved R_ILM1 50.2 mm to (175.4, 21.4), turned to 0 degrees
- moved C_IN2 50.1 mm to (171.8, 24.1), turned to 0 degrees
- moved C37 49.1 mm to (151.0, 40.0), turned to 0 degrees
- moved C35 48.9 mm to (150.5, 41.8), turned to 90 degrees
- moved U4 48.1 mm to (174.6, 23.9), turned to 0 degrees
- moved C_USB_BULK1 47.7 mm to (171.7, 26.5), turned to -90 degrees
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Connections:
- net Net-(U1-GPIO12) renamed /ADXL_DRDY
- J_OUT1 pad 2: unconnected-(J_OUT1-GND-Pad2) -> GND
- J_OUT1 pad 5: unconnected-(J_OUT1-SHIELD-Pad5) -> /SHIELD
- R22 pad 2: Net-(U1-GPIO20) -> Net-(U1-GPIO18)
- R27 pad 2: Net-(U3-*CS/SCL) -> /ADXL_CS
- U1 pad 12: Net-(U1-GPIO8) -> /ADXL_MISO
- U1 pad 13: Net-(U1-GPIO20) -> /ADXL_CS
- U1 pad 14: Net-(U1-GPIO10) -> /ADXL_SCLK
- U1 pad 15: Net-(U1-GPIO11) -> /ADXL_MOSI
- U1 pad 17: Net-(U1-GPIO13) -> /ADXL_INT2
- U1 pad 18: Net-(U1-GPIO14) -> /ADXL_INT1
- U1 pad 27: unconnected-(U1-GPIO16-Pad27) -> Net-(U1-GPIO16)
- U1 pad 28: unconnected-(U1-GPIO17-Pad28) -> Net-(U1-GPIO17)
- U1 pad 31: Net-(U1-GPIO19) -> unconnected-(U1-GPIO19-Pad31)
- U1 pad 32: Net-(U1-GPIO20) -> unconnected-(U1-GPIO20-Pad32)
- U2 pad 1: Net-(U1-GPIO18) -> Net-(U1-GPIO16)
- U2 pad 2: Net-(U1-GPIO20) -> Net-(U1-GPIO18)
- U2 pad 3: Net-(U1-GPIO20) -> Net-(U1-GPIO18)
- U2 pad 4: Net-(U1-GPIO19) -> Net-(U1-GPIO17)
- U3 pad 1: Net-(U3-*CS/SCL) -> /ADXL_CS
- U3 pad 12: Net-(U1-GPIO13) -> /ADXL_INT1
- U3 pad 13: Net-(U1-GPIO14) -> /ADXL_INT2
- U3 pad 2: Net-(U3-SCLK/VSSIO) -> /ADXL_SCLK
- U3 pad 3: Net-(U3-MOSI/SDA) -> /ADXL_MOSI
- U3 pad 4: Net-(U3-MISO/ASEL) -> /ADXL_MISO
Routing:
- net GND: track 118.0 -> 91.0 mm, vias 14 -> 13
- net Net-(U1-GPIO18): track 23.5 -> 0.00 mm
- net /3V3_DIG: track 30.2 -> 6.96 mm
- net /RS485_B: track 29.4 -> 6.35 mm
- net Net-(U1-GPIO20): track 21.8 -> 0.00 mm
- net /5V_SYS: track 21.8 -> 39.6 mm
- net Net-(U1-GPIO19): track 16.3 -> 0.00 mm
- net /USB_VBUS: track 27.6 -> 15.7 mm, vias 3 -> 2
- net /RS485_A: track 22.8 -> 11.3 mm
- net /USB DN: track 12.7 -> 6.20 mm
- net /USB DP: track 10.1 -> 3.66 mm
- net Net-(U1-QSPI_SD3): track 15.4 -> 21.5 mm
- net Net-(U1-QSPI_SCLK): track 13.4 -> 18.9 mm
- net Net-(U1-QSPI_SD0): track 10.6 -> 15.4 mm
- net Net-(JP1-B): track 4.52 -> 0.00 mm
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Other:
- board size 145.6 x 52 mm -> 145.2 x 84.4 mm
