File: hardware/KiCad - node V2/RP2350.kicad_sch (KiCad schematic)
At the start: 87 parts, among them J3 USB_C_Receptacle_USB2.0_14P, SW1 BOOTSEL, U1 RP2350A, U2 THVD1450DR, U3 ADXL355BEZ-RL7, U4 TPS2121RUXR, U5 USBLC6-2SC6, U6 TLV75733PDBVR, U7 W25Q128JVS, U8 TPS7A2033PDBVR

Commit message: Integrate node hardware and host tooling updates
Parts:
- C29: value 1uF -> 10uF
Changed lines of the file:
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@@
 			)
 		)
-		(property "Value" "1uF"
+		(property "Value" "10uF"
 			(at 147.3263 92.71 90)
 			(show_name no)
